File: 5v_reg.sch (KiCad schematic (older format))
At the start: 2 parts, among them U2 EHHD015A0A

Commit message: assign footprints to components
Parts:
- C4: footprint (none) -> Capacitors_SMD:C_0603
- U2: footprint (none) -> pdb:EHHD015A0A
Changed lines of the file:
@@
 F 0 "U2" H 5800 4250 60  0000 C CNN
 F 1 "EHHD015A0A" H 6000 3350 60  0000 C CNN
-F 2 "" H 5800 3750 60  0001 C CNN
+F 2 "pdb:EHHD015A0A" H 5800 3750 60  0001 C CNN
 F 3 "" H 5800 3750 60  0001 C CNN
 	1    6100 3800
@@
 F 0 "C4" H 5075 4050 50  0000 L CNN
 F 1 "100μ" H 5075 3850 50  0000 L CNN
-F 2 "" H 5088 3800 50  0001 C CNN
+F 2 "Capacitors_SMD:C_0603" H 5088 3800 50  0001 C CNN
 F 3 "" H 5050 3950 50  0001 C CNN
 	1    5050 3950
