File: input_power_switch.sch (KiCad schematic (older format))
At the start: 0 parts

Commit message: add input power switching circuit
Parts:
- added 0.002: R_Shunt, symbol R_Shunt
- added C?: C, symbol C
- added C? (x2): 1μ, symbol C
- added D? (x3): 50V, symbol D
- added L?: 1m, symbol L
- added Q? (x4): Q_NMOS_SSSGD, symbol Q_NMOS_SSSGD
- added U?: LTC1473, Housings_SSOP:SSOP-16_3.9x4.9mm_Pitch0.635mm, symbol LTC1473
Connections:
- new net: Q?.1 (S), Q?.1 (S), Q?.2 (S), Q?.3 (S), Q?.3 (S), U?.10 (SAB2)
- new net: Q?.4 (G), U?.11 (GA2)
- new net: 0.002.2, U?.12 (SENSE-)
- new net: 0.002.3, U?.13 (SENSE+)
- new net: Q?.4 (G), U?.14 (GB1)
- new net: Q?.1 (S), Q?.1 (S), Q?.2 (S), Q?.3 (S), Q?.3 (S), U?.15 (SAB1)
- new net: Q?.4 (G), U?.16 (GA1)
- new net: C?.1, U?.4 (TIMER)
- new net: C?.1, D?.1 (K), D?.1 (K), D?.1 (K), L?.1, U?.5 (V+)
- new net: C?.1, U?.6 (VGG)
- new net: L?.2, U?.7 (SW)
- new net: Q?.4 (G), U?.9 (GB2)
- new net: 0.002.4, Q?.5 (D), Q?.5 (D)
- new net GND: C?.2, C?.2, C?.2, D?.2 (A), U?.1 (IN1), U?.2 (IN2), U?.3 (~DIODE), U?.8 (GND)
- new net PWR_IN_1: D?.2 (A), Q?.5 (D)
- new net PWR_IN_2: D?.2 (A), Q?.5 (D)
- new net PWR_OUT: 0.002.1
