File: input_power_switch.sch (KiCad schematic (older format))
At the start: 13 parts

Commit message: clean up after annotate
Parts:
- C1: renamed from C?; value C -> 47n
- R2: renamed from 0.002; value R_Shunt -> 0.002
- gave numbers to parts that had none: 11
Changed lines of the file:
@@
 $EndDescr
 $Comp
-L LTC1473 U?
+L LTC1473 U1
 U 1 1 595A3FD7
 P 5550 4150
-F 0 "U?" H 5350 4650 50  0000 C CNN
+F 0 "U1" H 5350 4650 50  0000 C CNN
 F 1 "LTC1473" H 5450 3550 50  0000 C CNN
 F 2 "Housings_SSOP:SSOP-16_3.9x4.9mm_Pitch0.635mm" H 6250 3450 50  0001 C CNN
@@
 $EndComp
 $Comp
-L GND #PWR?
+L GND #PWR8
 U 1 1 595A40B8
 P 5050 4750
-F 0 "#PWR?" H 5050 4500 50  0001 C CNN
+F 0 "#PWR8" H 5050 4500 50  0001 C CNN
 F 1 "GND" H 5050 4600 50  0000 C CNN
 F 2 "" H 5050 4750 50  0001 C CNN
@@
 	5050 4550 5150 4550
 $Comp
-L GND #PWR?
+L GND #PWR3
 U 1 1 595A40D4
 P 3650 5350
-F 0 "#PWR?" H 3650 5100 50  0001 C CNN
+F 0 "#PWR3" H 3650 5100 50  0001 C CNN
 F 1 "GND" H 3650 5200 50  0000 C CNN
 F 2 "" H 3650 5350 50  0001 C CNN
@@
 $EndComp
 $Comp
-L C C?
+L C C1
 U 1 1 595A40ED
 P 3650 4900
-F 0 "C?" H 3675 5000 50  0000 L CNN
-F 1 "C" H 3675 4800 50  0000 L CNN
+F 0 "C1" H 3675 5000 50  0000 L CNN
+F 1 "47n" H 3675 4800 50  0000 L CNN
 F 2 "" H 3688 4750 50  0001 C CNN
 F 3 "" H 3650 4900 50  0001 C CNN
@@
 	3650 5350 3650 5050
 $Comp
-L L L?
+L L L1
 U 1 1 595A448B
 P 4900 4450
-F 0 "L?" V 4850 4450 50  0000 C CNN
+F 0 "L1" V 4850 4450 50  0000 C CNN
 F 1 "1m" V 4975 4450 50  0000 C CNN
 F 2 "" H 4900 4450 50  0001 C CNN
@@
 $EndComp
 $Comp
-L C C?
+L C C2
 U 1 1 595A4651
 P 3950 4900
-F 0 "C?" H 3975 5000 50  0000 L CNN
+F 0 "C2" H 3975 5000 50  0000 L CNN
 F 1 "1μ" H 3975 4800 50  0000 L CNN
 F 2 "" H 3988 4750 50  0001 C CNN
@@
 	3950 4750 3950 4350
 $Comp
-L GND #PWR?
+L GND #PWR4
 U 1 1 595A499D
 P 3950 5350
-F 0 "#PWR?" H 3950 5100 50  0001 C CNN
+F 0 "#PWR4" H 3950 5100 50  0001 C CNN
 F 1 "GND" H 3950 5200 50  0000 C CNN
 F 2 "" H 3950 5350 50  0001 C CNN
@@
 	3950 5050 3950 5350
 $Comp
-L C C?
+L C C3
 U 1 1 595A4DC4
 P 4600 4900
-F 0 "C?" H 4625 5000 50  0000 L CNN
+F 0 "C3" H 4625 5000 50  0000 L CNN
 F 1 "1μ" H 4625 4800 50  0000 L CNN
 F 2 "" H 4638 4750 50  0001 C CNN
@@
 $EndComp
 $Comp
-L GND #PWR?
+L GND #PWR6
 U 1 1 595A4E35
 P 4600 5350
-F 0 "#PWR?" H 4600 5100 50  0001 C CNN
+F 0 "#PWR6" H 4600 5100 50  0001 C CNN
 F 1 "GND" H 4600 5200 50  0000 C CNN
 F 2 "" H 4600 5350 50  0001 C CNN
@@
 	4600 5050 4600 5350
 $Comp
-L D D?
+L D D3
 U 1 1 595A4FB7
 P 4300 4900
-F 0 "D?" H 4300 5000 50  0000 C CNN
+F 0 "D3" H 4300 5000 50  0000 C CNN
 F 1 "50V" H 4300 4800 50  0000 C CNN
 F 2 "" H 4300 4900 50  0001 C CNN
@@
 $EndComp
 $Comp
-L GND #PWR?
+L GND #PWR5
 U 1 1 595A5026
 P 4300 5350
-F 0 "#PWR?" H 4300 5100 50  0001 C CNN
+F 0 "#PWR5" H 4300 5100 50  0001 C CNN
 F 1 "GND" H 4300 5200 50  0000 C CNN
 F 2 "" H 4300 5350 50  0001 C CNN
@@
 	3650 4150 5150 4150
 $Comp
-L D D?
+L D D2
 U 1 1 595A71D4
 P 4100 3500
-F 0 "D?" H 4100 3600 50  0000 C CNN
+F 0 "D2" H 4100 3600 50  0000 C CNN
 F 1 "50V" H 4100 3400 50  0000 C CNN
 F 2 "" H 4100 3500 50  0001 C CNN
@@
 $EndComp
 $Comp
-L D D?
+L D D1
 U 1 1 595A723B
 P 3750 3500
-F 0 "D?" H 3750 3600 50  0000 C CNN
+F 0 "D1" H 3750 3600 50  0000 C CNN
 F 1 "50V" H 3750 3400 50  0000 C CNN
 F 2 "" H 3750 3500 50  0001 C CNN
@@
 	6150 3850 6050 3850
 $Comp
-L Q_NMOS_SSSGD Q?
+L Q_NMOS_SSSGD Q1
 U 1 1 595AC07D
 P 6150 2750
-F 0 "Q?" V 6450 2750 50  0000 L CNN
+F 0 "Q1" V 6450 2750 50  0000 L CNN
 F 1 "Q_NMOS_SSSGD" V 6350 2700 50  0001 L CNN
 F 2 "" H 6350 2850 50  0001 C CNN
@@
 $EndComp
 $Comp
-L Q_NMOS_SSSGD Q?
+L Q_NMOS_SSSGD Q2
 U 1 1 595AC083
 P 6850 2750
-F 0 "Q?" V 7150 2750 50  0000 L CNN
+F 0 "Q2" V 7150 2750 50  0000 L CNN
 F 1 "Q_NMOS_SSSGD" H 7050 2700 50  0001 L CNN
 F 2 "" H 7050 2850 50  0001 C CNN
@@
 	6850 2950 6850 4050
 $Comp
-L Q_NMOS_SSSGD Q?
+L Q_NMOS_SSSGD Q3
 U 1 1 595B1F56
 P 7300 3300
-F 0 "Q?" V 7600 3300 50  0000 L CNN
+F 0 "Q3" V 7600 3300 50  0000 L CNN
 F 1 "Q_NMOS_SSSGD" V 7500 3250 50  0001 L CNN
 F 2 "" H 7500 3400 50  0001 C CNN
@@
 $EndComp
 $Comp
-L Q_NMOS_SSSGD Q?
+L Q_NMOS_SSSGD Q4
 U 1 1 595B1F5C
 P 8000 3300
-F 0 "Q?" V 8300 3300 50  0000 L CNN
+F 0 "Q4" V 8300 3300 50  0000 L CNN
 F 1 "Q_NMOS_SSSGD" H 8200 3250 50  0001 L CNN
 F 2 "" H 8200 3400 50  0001 C CNN
@@
 Connection ~ 3750 2650
 $Comp
-L R_Shunt 0.002
+L R_Shunt R2
 U 1 1 595B8397
 P 8950 2900
-F 0 "0.002" V 8850 2900 50  0000 C CNN
-F 1 "R_Shunt" V 8850 2900 50  0001 C CNN
+F 0 "R2" V 8850 2900 50  0000 C CNN
+F 1 "0.002" V 8950 2900 50  0000 C CNN
 F 2 "" V 8880 2900 50  0001 C CNN
 F 3 "" H 8950 2900 50  0001 C CNN
@@
 	9050 4250 6050 4250
 $Comp
-L GND #PWR?
+L GND #PWR7
 U 1 1 595C41E9
 P 4900 3950
-F 0 "#PWR?" H 4900 3700 50  0001 C CNN
+F 0 "#PWR7" H 4900 3700 50  0001 C CNN
 F 1 "GND" H 4900 3800 50  0000 C CNN
 F 2 "" H 4900 3950 50  0001 C CNN

Commit message: fix broken annotation
Parts:
- U1: symbol LTC1473 -> LTC1473-RESCUE-pdb
Changed lines of the file:
@@
 EESchema Schematic File Version 2
+LIBS:pdb-rescue
 LIBS:power
 LIBS:device
@@
 $EndDescr
 $Comp
-L LTC1473 U1
+L LTC1473-RESCUE-pdb U1
 U 1 1 595A3FD7
 P 5550 4150
+AR Path="/595A3FD7" Ref="U1"  Part="1"
+AR Path="/5957A7A6/595A3FD7" Ref="U1"  Part="1"
 F 0 "U1" H 5350 4650 50  0000 C CNN
 F 1 "LTC1473" H 5450 3550 50  0000 C CNN

Commit message: fix issue with incorrect symbol
Parts:
- removed U1: LTC1473, Housings_SSOP:SSOP-16_3.9x4.9mm_Pitch0.635mm, symbol LTC1473-RESCUE-pdb
- added U1: LTC1473, Housings_SSOP:SSOP-16_3.9x4.9mm_Pitch0.635mm, symbol LTC1473
Connections:
- net GND: now also U1.1 (IN1), U1.2 (IN2), U1.3 (~DIODE), U1.8 (GND)
- net at Q3.1 (S), Q3.3 (S), Q4.1 (S)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: now also U1.10 (SAB2)
- net at Q3.4 (G): now also U1.11 (GA2)
- net at R2.2: now also U1.12 (SENSE-)
- net at R2.3: now also U1.13 (SENSE+)
- net at Q2.4 (G): now also U1.14 (GB1)
- net at Q1.1 (S), Q1.3 (S), Q2.1 (S)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: now also U1.15 (SAB1)
- net at Q1.4 (G): now also U1.16 (GA1)
- net at C1.1: now also U1.4 (TIMER)
- net at C3.1, D1.1 (K), D2.1 (K)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: now also U1.5 (V+)
- net at C2.1: now also U1.6 (VGG)
- net at L1.2: now also U1.7 (SW)
- net at Q4.4 (G): now also U1.9 (GB2)
Changed lines of the file:
@@
 $EndDescr
 $Comp
-L LTC1473-RESCUE-pdb U1
-U 1 1 595A3FD7
-P 5550 4150
-AR Path="/595A3FD7" Ref="U1"  Part="1"
-AR Path="/5957A7A6/595A3FD7" Ref="U1"  Part="1"
-F 0 "U1" H 5350 4650 50  0000 C CNN
-F 1 "LTC1473" H 5450 3550 50  0000 C CNN
-F 2 "Housings_SSOP:SSOP-16_3.9x4.9mm_Pitch0.635mm" H 6250 3450 50  0001 C CNN
-F 3 "./datasheets/ltc1473.pdf" H 5350 4650 50  0001 C CNN
-	1    5550 4150
-	1    0    0    -1
-$EndComp
-$Comp
-L GND #PWR8
+L GND #PWR03
 U 1 1 595A40B8
 P 5050 4750
-F 0 "#PWR8" H 5050 4500 50  0001 C CNN
+F 0 "#PWR03" H 5050 4500 50  0001 C CNN
 F 1 "GND" H 5050 4600 50  0000 C CNN
 F 2 "" H 5050 4750 50  0001 C CNN
@@
 	5050 4550 5150 4550
 $Comp
-L GND #PWR3
+L GND #PWR04
 U 1 1 595A40D4
 P 3650 5350
-F 0 "#PWR3" H 3650 5100 50  0001 C CNN
+F 0 "#PWR04" H 3650 5100 50  0001 C CNN
 F 1 "GND" H 3650 5200 50  0000 C CNN
 F 2 "" H 3650 5350 50  0001 C CNN
@@
 	3950 4750 3950 4350
 $Comp
-L GND #PWR4
+L GND #PWR05
 U 1 1 595A499D
 P 3950 5350
-F 0 "#PWR4" H 3950 5100 50  0001 C CNN
+F 0 "#PWR05" H 3950 5100 50  0001 C CNN
 F 1 "GND" H 3950 5200 50  0000 C CNN
 F 2 "" H 3950 5350 50  0001 C CNN
@@
 $EndComp
 $Comp
-L GND #PWR6
+L GND #PWR06
 U 1 1 595A4E35
 P 4600 5350
-F 0 "#PWR6" H 4600 5100 50  0001 C CNN
+F 0 "#PWR06" H 4600 5100 50  0001 C CNN
 F 1 "GND" H 4600 5200 50  0000 C CNN
 F 2 "" H 4600 5350 50  0001 C CNN
@@
 $EndComp
 $Comp
-L GND #PWR5
+L GND #PWR07
 U 1 1 595A5026
 P 4300 5350
-F 0 "#PWR5" H 4300 5100 50  0001 C CNN
+F 0 "#PWR07" H 4300 5100 50  0001 C CNN
 F 1 "GND" H 4300 5200 50  0000 C CNN
 F 2 "" H 4300 5350 50  0001 C CNN
@@
 	9050 4250 6050 4250
 $Comp
-L GND #PWR7
+L GND #PWR08
 U 1 1 595C41E9
 P 4900 3950
-F 0 "#PWR7" H 4900 3700 50  0001 C CNN
+F 0 "#PWR08" H 4900 3700 50  0001 C CNN
 F 1 "GND" H 4900 3800 50  0000 C CNN
 F 2 "" H 4900 3950 50  0001 C CNN
@@
 	4900 3950 5150 3950
 Connection ~ 5100 3950
+$Comp
+L LTC1473 U1
+U 1 1 59624468
+P 5550 4150
+F 0 "U1" H 5350 4650 50  0000 C CNN
+F 1 "LTC1473" H 5450 3550 50  0000 C CNN
+F 2 "Housings_SSOP:SSOP-16_3.9x4.9mm_Pitch0.635mm" H 6250 3450 50  0001 C CNN
+F 3 "" H 5350 4650 50  0001 C CNN
+	1    5550 4150
+	1    0    0    -1
+$EndComp
 $EndSCHEMATC
