File: input_power_switch.sch (KiCad schematic (older format))
At the start: 13 parts, among them Q1 Q_NMOS_SSSGD, Q2 Q_NMOS_SSSGD, Q3 Q_NMOS_SSSGD, Q4 Q_NMOS_SSSGD, U1 LTC1473

Commit message: assign footprints to components
Parts:
- C1, C2, C3: footprint (none) -> Capacitors_SMD:C_0603
- D1, D2, D3: footprint (none) -> Diodes_SMD:D_SMA
- L1: footprint (none) -> Inductors_SMD:L_0805
- Q1, Q2, Q3, Q4: footprint (none) -> TO_SOT_Packages_SMD:SOT-669_LFPAK
- R2: footprint (none) -> pdb:WSLP2726
Changed lines of the file:
@@
 F 0 "C1" H 3675 5000 50  0000 L CNN
 F 1 "47n" H 3675 4800 50  0000 L CNN
-F 2 "" H 3688 4750 50  0001 C CNN
+F 2 "Capacitors_SMD:C_0603" H 3688 4750 50  0001 C CNN
 F 3 "" H 3650 4900 50  0001 C CNN
 	1    3650 4900
@@
 F 0 "L1" V 4850 4450 50  0000 C CNN
 F 1 "1m" V 4975 4450 50  0000 C CNN
-F 2 "" H 4900 4450 50  0001 C CNN
+F 2 "Inductors_SMD:L_0805" H 4900 4450 50  0001 C CNN
 F 3 "" H 4900 4450 50  0001 C CNN
 	1    4900 4450
@@
 F 0 "C2" H 3975 5000 50  0000 L CNN
 F 1 "1μ" H 3975 4800 50  0000 L CNN
-F 2 "" H 3988 4750 50  0001 C CNN
+F 2 "Capacitors_SMD:C_0603" H 3988 4750 50  0001 C CNN
 F 3 "" H 3950 4900 50  0001 C CNN
 	1    3950 4900
@@
 F 0 "C3" H 4625 5000 50  0000 L CNN
 F 1 "1μ" H 4625 4800 50  0000 L CNN
-F 2 "" H 4638 4750 50  0001 C CNN
+F 2 "Capacitors_SMD:C_0603" H 4638 4750 50  0001 C CNN
 F 3 "" H 4600 4900 50  0001 C CNN
 	1    4600 4900
@@
 F 0 "D3" H 4300 5000 50  0000 C CNN
 F 1 "50V" H 4300 4800 50  0000 C CNN
-F 2 "" H 4300 4900 50  0001 C CNN
+F 2 "Diodes_SMD:D_SMA" H 4300 4900 50  0001 C CNN
 F 3 "" H 4300 4900 50  0001 C CNN
 	1    4300 4900
@@
 F 0 "D2" H 4100 3600 50  0000 C CNN
 F 1 "50V" H 4100 3400 50  0000 C CNN
-F 2 "" H 4100 3500 50  0001 C CNN
+F 2 "Diodes_SMD:D_SMA" H 4100 3500 50  0001 C CNN
 F 3 "" H 4100 3500 50  0001 C CNN
 	1    4100 3500
@@
 F 0 "D1" H 3750 3600 50  0000 C CNN
 F 1 "50V" H 3750 3400 50  0000 C CNN
-F 2 "" H 3750 3500 50  0001 C CNN
+F 2 "Diodes_SMD:D_SMA" H 3750 3500 50  0001 C CNN
 F 3 "" H 3750 3500 50  0001 C CNN
 	1    3750 3500
@@
 F 0 "Q1" V 6450 2750 50  0000 L CNN
 F 1 "Q_NMOS_SSSGD" V 6350 2700 50  0001 L CNN
-F 2 "" H 6350 2850 50  0001 C CNN
+F 2 "TO_SOT_Packages_SMD:SOT-669_LFPAK" H 6350 2850 50  0001 C CNN
 F 3 "" H 6150 2750 50  0001 C CNN
 	1    6150 2750
@@
 F 0 "Q2" V 7150 2750 50  0000 L CNN
 F 1 "Q_NMOS_SSSGD" H 7050 2700 50  0001 L CNN
-F 2 "" H 7050 2850 50  0001 C CNN
+F 2 "TO_SOT_Packages_SMD:SOT-669_LFPAK" H 7050 2850 50  0001 C CNN
 F 3 "" H 6850 2750 50  0001 C CNN
 	1    6850 2750
@@
 F 0 "Q3" V 7600 3300 50  0000 L CNN
 F 1 "Q_NMOS_SSSGD" V 7500 3250 50  0001 L CNN
-F 2 "" H 7500 3400 50  0001 C CNN
+F 2 "TO_SOT_Packages_SMD:SOT-669_LFPAK" H 7500 3400 50  0001 C CNN
 F 3 "" H 7300 3300 50  0001 C CNN
 	1    7300 3300
@@
 F 0 "Q4" V 8300 3300 50  0000 L CNN
 F 1 "Q_NMOS_SSSGD" H 8200 3250 50  0001 L CNN
-F 2 "" H 8200 3400 50  0001 C CNN
+F 2 "TO_SOT_Packages_SMD:SOT-669_LFPAK" H 8200 3400 50  0001 C CNN
 F 3 "" H 8000 3300 50  0001 C CNN
 	1    8000 3300
@@
 F 0 "R2" V 8850 2900 50  0000 C CNN
 F 1 "0.002" V 8950 2900 50  0000 C CNN
-F 2 "" V 8880 2900 50  0001 C CNN
+F 2 "pdb:WSLP2726" V 8880 2900 50  0001 C CNN
 F 3 "" H 8950 2900 50  0001 C CNN
 	1    8950 2900
