File: killswitch.sch (KiCad schematic (older format))
At the start: 0 parts

Commit message: add killswitch
Parts:
- added 10k: R, symbol R
- added C?: 0.1μ, symbol C
- added U?: A1120, symbol A1120
Connections:
- new net GND: C?.2, U?.3 (GND)
- new net PWR_ENABLE: 10k.2, U?.2 (VOUT)
- new net PWR_IN: 10k.1, C?.1, U?.1 (VCC)
Changed lines of the file:
@@
 LIBS:nmos_sssgd
 LIBS:ehhd015a0a
+LIBS:a1120
 LIBS:pdb-cache
 EELAYER 25 0
@@
 Comment4 ""
 $EndDescr
+$Comp
+L A1120 U?
+U 1 1 595CBD70
+P 6050 4000
+F 0 "U?" H 5850 4300 60  0000 C CNN
+F 1 "A1120" H 5950 3700 60  0000 C CNN
+F 2 "" H 5950 4000 60  0001 C CNN
+F 3 "" H 5950 4000 60  0001 C CNN
+	1    6050 4000
+	1    0    0    -1
+$EndComp
+$Comp
+L C C?
+U 1 1 595CBDEE
+P 5250 4200
+F 0 "C?" H 5275 4300 50  0000 L CNN
+F 1 "0.1μ" H 5275 4100 50  0000 L CNN
+F 2 "" H 5288 4050 50  0001 C CNN
+F 3 "" H 5250 4200 50  0001 C CNN
+	1    5250 4200
+	1    0    0    -1
+$EndComp
+$Comp
+L GND #PWR?
+U 1 1 595CBE78
+P 5250 4450
+F 0 "#PWR?" H 5250 4200 50  0001 C CNN
+F 1 "GND" H 5250 4300 50  0000 C CNN
+F 2 "" H 5250 4450 50  0001 C CNN
+F 3 "" H 5250 4450 50  0001 C CNN
+	1    5250 4450
+	1    0    0    -1
+$EndComp
+Wire Wire Line
+	5250 4350 5250 4450
+Wire Wire Line
+	5250 3500 5250 4050
+$Comp
+L GND #PWR?
+U 1 1 595CBF79
+P 5550 4450
+F 0 "#PWR?" H 5550 4200 50  0001 C CNN
+F 1 "GND" H 5550 4300 50  0000 C CNN
+F 2 "" H 5550 4450 50  0001 C CNN
+F 3 "" H 5550 4450 50  0001 C CNN
+	1    5550 4450
+	1    0    0    -1
+$EndComp
+Wire Wire Line
+	5650 4100 5550 4100
+Wire Wire Line
+	5550 4100 5550 4450
+Wire Wire Line
+	5250 3900 5650 3900
+$Comp
+L R 10k
+U 1 1 595CC072
+P 6550 3750
+F 0 "10k" V 6630 3750 50  0000 C CNN
+F 1 "R" V 6550 3750 50  0000 C CNN
+F 2 "" V 6480 3750 50  0001 C CNN
+F 3 "" H 6550 3750 50  0001 C CNN
+	1    6550 3750
+	1    0    0    -1
+$EndComp
+Wire Wire Line
+	6450 4000 6850 4000
+Wire Wire Line
+	6550 3900 6550 4000
+Connection ~ 6550 4000
+Text HLabel 6850 4000 2    60   Output ~ 0
+PWR_ENABLE
+Text HLabel 4650 3500 0    60   Input ~ 0
+PWR_IN
+Wire Wire Line
+	4650 3500 6550 3500
+Wire Wire Line
+	6550 3500 6550 3600
+Connection ~ 5250 3500
+Connection ~ 5250 3900
+Text Label 5250 3500 2    60   ~ 0
+5V
 $EndSCHEMATC
