File: killswitch.sch (KiCad schematic (older format))
At the start: 3 parts, among them U9 A1120

Commit message: assign footprints to components
Parts:
- C9: footprint (none) -> Capacitors_SMD:C_0603
- R3: footprint (none) -> Resistors_SMD:R_0603
- U9: footprint (none) -> Connectors_Molex:Molex_KK-6410-03_03x2.54mm_Straight
Changed lines of the file:
@@
 F 0 "C9" H 5275 4300 50  0000 L CNN
 F 1 "0.1μ" H 5275 4100 50  0000 L CNN
-F 2 "" H 5288 4050 50  0001 C CNN
+F 2 "Capacitors_SMD:C_0603" H 5288 4050 50  0001 C CNN
 F 3 "" H 5250 4200 50  0001 C CNN
 	1    5250 4200
@@
 F 0 "R3" V 6630 3750 50  0000 C CNN
 F 1 "10k" V 6550 3750 50  0000 C CNN
-F 2 "" V 6480 3750 50  0001 C CNN
+F 2 "Resistors_SMD:R_0603" V 6480 3750 50  0001 C CNN
 F 3 "" H 6550 3750 50  0001 C CNN
 	1    6550 3750
@@
 F 0 "U9" H 5850 4300 50  0000 C CNN
 F 1 "A1120" H 5950 3700 50  0000 C CNN
-F 2 "" H 5950 4000 50  0001 C CNN
+F 2 "Connectors_Molex:Molex_KK-6410-03_03x2.54mm_Straight" H 5950 4000 50  0001 C CNN
 F 3 "" H 5950 4000 50  0001 C CNN
 	1    6050 4000
