File: 5v_power_switch_A.sch (KiCad schematic (older format))
At the start: 6 parts, among them U4 74HC14, U7 TPS2024D

Commit message: assign footprints to components
Parts:
- C5, C7: footprint (none) -> Capacitors_SMD:C_0603
- D6: footprint (none) -> LEDs:LED_0805
- R6: footprint (none) -> Resistors_SMD:R_0603
- U4: footprint (none) -> Housings_SSOP:SSOP-14_5.3x6.2mm_Pitch0.65mm
- U7: footprint (none) -> Housings_SOIC:SOIC-8_3.9x4.9mm_Pitch1.27mm
Changed lines of the file:
@@
 F 0 "C5" H 5675 3700 50  0000 L CNN
 F 1 "0.1μ" H 5675 3500 50  0000 L CNN
-F 2 "" H 5688 3450 50  0001 C CNN
+F 2 "Capacitors_SMD:C_0603" H 5688 3450 50  0001 C CNN
 F 3 "" H 5650 3600 50  0001 C CNN
 	1    5650 3600
@@
 F 0 "U4" H 5250 3400 50  0000 C CNN
 F 1 "74HC14" H 5300 3200 50  0000 C CNN
-F 2 "" H 5100 3300 50  0001 C CNN
+F 2 "Housings_SSOP:SSOP-14_5.3x6.2mm_Pitch0.65mm" H 5100 3300 50  0001 C CNN
 F 3 "" H 5100 3300 50  0001 C CNN
 	1    5100 3300
@@
 F 0 "U7" H 6300 3800 50  0000 C CNN
 F 1 "TPS2024D" H 6400 2800 50  0000 C CNN
-F 2 "" H 7600 2400 50  0001 C CNN
+F 2 "Housings_SOIC:SOIC-8_3.9x4.9mm_Pitch1.27mm" H 7600 2400 50  0001 C CNN
 F 3 "" H 7600 2400 50  0001 C CNN
 	1    6500 3300
@@
 F 0 "R6" V 7330 3250 50  0000 C CNN
 F 1 "1k5" V 7250 3250 50  0000 C CNN
-F 2 "" V 7180 3250 50  0001 C CNN
+F 2 "Resistors_SMD:R_0603" V 7180 3250 50  0001 C CNN
 F 3 "" H 7250 3250 50  0001 C CNN
 	1    7250 3250
@@
 F 0 "D6" H 7250 3700 50  0000 C CNN
 F 1 "LED" H 7250 3500 50  0000 C CNN
-F 2 "" H 7250 3600 50  0001 C CNN
+F 2 "LEDs:LED_0805" H 7250 3600 50  0001 C CNN
 F 3 "" H 7250 3600 50  0001 C CNN
 	1    7250 3600
@@
 F 0 "U4" H 5250 4600 50  0000 C CNN
 F 1 "74HC14" H 5300 4400 50  0000 C CNN
-F 2 "" H 5100 4500 50  0001 C CNN
+F 2 "Housings_SSOP:SSOP-14_5.3x6.2mm_Pitch0.65mm" H 5100 4500 50  0001 C CNN
 F 3 "" H 5100 4500 50  0001 C CNN
 	2    5100 4500
@@
 F 0 "U4" H 5250 5150 50  0000 C CNN
 F 1 "74HC14" H 5300 4950 50  0000 C CNN
-F 2 "" H 5100 5050 50  0001 C CNN
+F 2 "Housings_SSOP:SSOP-14_5.3x6.2mm_Pitch0.65mm" H 5100 5050 50  0001 C CNN
 F 3 "" H 5100 5050 50  0001 C CNN
 	3    5100 5050
@@
 F 0 "U4" H 5250 5500 50  0000 C CNN
 F 1 "74HC14" H 5300 5300 50  0000 C CNN
-F 2 "" H 5100 5400 50  0001 C CNN
+F 2 "Housings_SSOP:SSOP-14_5.3x6.2mm_Pitch0.65mm" H 5100 5400 50  0001 C CNN
 F 3 "" H 5100 5400 50  0001 C CNN
 	4    5100 5400
@@
 F 0 "U4" H 5250 5850 50  0000 C CNN
 F 1 "74HC14" H 5300 5650 50  0000 C CNN
-F 2 "" H 5100 5750 50  0001 C CNN
+F 2 "Housings_SSOP:SSOP-14_5.3x6.2mm_Pitch0.65mm" H 5100 5750 50  0001 C CNN
 F 3 "" H 5100 5750 50  0001 C CNN
 	5    5100 5750
@@
 F 0 "C6" H 4375 4600 50  0000 L CNN
 F 1 "0.1μ" H 4375 4400 50  0000 L CNN
-F 2 "" H 4388 4350 50  0001 C CNN
+F 2 "Capacitors_SMD:C_0603" H 4388 4350 50  0001 C CNN
 F 3 "" H 4350 4500 50  0001 C CNN
 	1    4350 4500
