File: 5v_power_switch_B.sch (KiCad schematic (older format))
At the start: 5 parts, among them U4 74HC14, U5 TPS2024D

Commit message: assign footprints to components
Parts:
- C7: footprint (none) -> Capacitors_SMD:C_0603
- D8: footprint (none) -> LEDs:LED_0805
- R8: footprint (none) -> Resistors_SMD:R_0603
- U4: footprint (none) -> Housings_SSOP:SSOP-14_5.3x6.2mm_Pitch0.65mm
- U5: footprint (none) -> Housings_SOIC:SOIC-8_3.9x4.9mm_Pitch1.27mm
Changed lines of the file:
@@
 F 0 "C7" H 5325 3900 50  0000 L CNN
 F 1 "0.1μ" H 5325 3700 50  0000 L CNN
-F 2 "" H 5338 3650 50  0001 C CNN
+F 2 "Capacitors_SMD:C_0603" H 5338 3650 50  0001 C CNN
 F 3 "" H 5300 3800 50  0001 C CNN
 	1    5300 3800
@@
 F 0 "U4" H 4900 3600 50  0000 C CNN
 F 1 "74HC14" H 4950 3400 50  0000 C CNN
-F 2 "" H 4750 3500 50  0001 C CNN
+F 2 "Housings_SSOP:SSOP-14_5.3x6.2mm_Pitch0.65mm" H 4750 3500 50  0001 C CNN
 F 3 "" H 4750 3500 50  0001 C CNN
 	6    4750 3500
@@
 F 0 "U5" H 5950 4000 50  0000 C CNN
 F 1 "TPS2024D" H 6050 3000 50  0000 C CNN
-F 2 "" H 7250 2600 50  0001 C CNN
+F 2 "Housings_SOIC:SOIC-8_3.9x4.9mm_Pitch1.27mm" H 7250 2600 50  0001 C CNN
 F 3 "" H 7250 2600 50  0001 C CNN
 	1    6150 3500
@@
 F 0 "R8" V 6980 3450 50  0000 C CNN
 F 1 "1k5" V 6900 3450 50  0000 C CNN
-F 2 "" V 6830 3450 50  0001 C CNN
+F 2 "Resistors_SMD:R_0603" V 6830 3450 50  0001 C CNN
 F 3 "" H 6900 3450 50  0001 C CNN
 	1    6900 3450
@@
 F 0 "D8" H 6900 3900 50  0000 C CNN
 F 1 "LED" H 6900 3700 50  0000 C CNN
-F 2 "" H 6900 3800 50  0001 C CNN
+F 2 "LEDs:LED_0805" H 6900 3800 50  0001 C CNN
 F 3 "" H 6900 3800 50  0001 C CNN
 	1    6900 3800
